File: 555_pwm/555_pwm.kicad_sch (KiCad schematic)
At the start: 2 parts, among them U1 NE555D

Commit message: aaa
Parts:
- added C2: C, symbol Device:C
- added R1, R2: R, symbol Device:R
Connections:
- net at C1.1: now also U1.2 (TR), U1.6 (THR), C2.2, R2.2
- net GND: now reaches U1.1 (GND)
- net GND: now also C2.1
- net +5V: now reaches U1.4 (R)
- net +5V: now also U1.8 (VCC), R1.1
- net at U1.7 (DIS): now also R1.2, R2.1
Changed lines of the file:
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@@
 (kicad_sch (version 20230121) (generator eeschema)
   (paper "A4")
+  (junction (at 127 60.96) (diameter 0) (color 0 0 0 0)
+  )
+  (junction (at 96.52 77.47) (diameter 0) (color 0 0 0 0)
+  )
+  (junction (at 139.7 82.55) (diameter 0) (color 0 0 0 0)
+  )
+  (junction (at 147.32 77.47) (diameter 0) (color 0 0 0 0)
+  )
+  (junction (at 139.7 88.9) (diameter 0) (color 0 0 0 0)
+  )
+  (junction (at 127 88.9) (diameter 0) (color 0 0 0 0)
+  )
+  (wire (pts (xy 139.7 82.55) (xy 139.7 88.9))
+    (stroke (width 0) (type default))
+  )
+  (wire (pts (xy 96.52 72.39) (xy 96.52 77.47))
+    (stroke (width 0) (type default))
+  )
+  (wire (pts (xy 114.3 72.39) (xy 96.52 72.39))
+    (stroke (width 0) (type default))
+  )
+  (wire (pts (xy 147.32 77.47) (xy 147.32 82.55))
+    (stroke (width 0) (type default))
+  )
+  (wire (pts (xy 127 87.63) (xy 127 88.9))
+    (stroke (width 0) (type default))
+  )
+  (wire (pts (xy 127 60.96) (xy 127 67.31))
+    (stroke (width 0) (type default))
+  )
+  (wire (pts (xy 127 88.9) (xy 127 99.06))
+    (stroke (width 0) (type default))
+  )
+  (wire (pts (xy 127 88.9) (xy 132.08 88.9))
+    (stroke (width 0) (type default))
+  )
+  (wire (pts (xy 99.06 60.96) (xy 99.06 82.55))
+    (stroke (width 0) (type default))
+  )
+  (wire (pts (xy 147.32 60.96) (xy 134.62 60.96))
+    (stroke (width 0) (type default))
+  )
+  (wire (pts (xy 147.32 77.47) (xy 147.32 60.96))
+    (stroke (width 0) (type default))
+  )
+  (wire (pts (xy 96.52 77.47) (xy 106.68 77.47))
+    (stroke (width 0) (type default))
+  )
+  (wire (pts (xy 96.52 77.47) (xy 96.52 93.98))
+    (stroke (width 0) (type default))
+  )
+  (wire (pts (xy 99.06 60.96) (xy 127 60.96))
+    (stroke (width 0) (type default))
+  )
+  (wire (pts (xy 139.7 88.9) (xy 139.7 93.98))
+    (stroke (width 0) (type default))
+  )
+  (wire (pts (xy 96.52 93.98) (xy 139.7 93.98))
+    (stroke (width 0) (type default))
+  )
+  (wire (pts (xy 139.7 77.47) (xy 147.32 77.47))
+    (stroke (width 0) (type default))
+  )
+  (wire (pts (xy 114.3 82.55) (xy 99.06 82.55))
+    (stroke (width 0) (type default))
+  )
+  (wire (pts (xy 127 50.8) (xy 127 60.96))
+    (stroke (width 0) (type default))
+  )
+  (symbol (lib_id "power:+5V") (at 127 50.8 0) (unit 1)
+    (in_bom yes) (on_board yes) (dnp no) (fields_autoplaced)
+    (property "Reference" "#PWR01" (at 127 54.61 0)
+      (effects (font (size 1.27 1.27)) hide)
+    )
+    (property "Value" "+5V" (at 127 45.72 0)
+      (effects (font (size 1.27 1.27)))
+    )
+    (property "Footprint" "" (at 127 50.8 0)
+      (effects (font (size 1.27 1.27)) hide)
+    )
+    (property "Datasheet" "" (at 127 50.8 0)
+      (effects (font (size 1.27 1.27)) hide)
+    )
+    (pin "1")
+    (instances
+      (project "555_pwm"
+        (path "/76d5dda2-c124-4f87-b6ec-acef9f17eff7"
+          (reference "#PWR01") (unit 1)
+        )
+      )
+    )
+  )
+  (symbol (lib_id "Device:R") (at 130.81 60.96 90) (unit 1)
+    (in_bom yes) (on_board yes) (dnp no) (fields_autoplaced)
+    (property "Reference" "R1" (at 130.81 54.61 90)
+      (effects (font (size 1.27 1.27)))
+    )
+    (property "Value" "R" (at 130.81 57.15 90)
+      (effects (font (size 1.27 1.27)))
+    )
+    (property "Footprint" "" (at 130.81 62.738 90)
+      (effects (font (size 1.27 1.27)) hide)
+    )
+    (property "Datasheet" "~" (at 130.81 60.96 0)
+      (effects (font (size 1.27 1.27)) hide)
+    )
+    (pin "1")
+    (pin "2")
+    (instances
+      (project "555_pwm"
+        (path "/76d5dda2-c124-4f87-b6ec-acef9f17eff7"
+          (reference "R1") (unit 1)
+        )
+      )
+    )
+  )
+  (symbol (lib_id "Device:R") (at 143.51 82.55 270) (unit 1)
+    (in_bom yes) (on_board yes) (dnp no)
+    (property "Reference" "R2" (at 143.51 76.2 90)
+      (effects (font (size 1.27 1.27)))
+    )
+    (property "Value" "R" (at 143.51 78.74 90)
+      (effects (font (size 1.27 1.27)))
+    )
+    (property "Footprint" "" (at 143.51 80.772 90)
+      (effects (font (size 1.27 1.27)) hide)
+    )
+    (property "Datasheet" "~" (at 143.51 82.55 0)
+      (effects (font (size 1.27 1.27)) hide)
+    )
+    (pin "1")
+    (pin "2")
+    (instances
+      (project "555_pwm"
+        (path "/76d5dda2-c124-4f87-b6ec-acef9f17eff7"
+          (reference "R2") (unit 1)
+        )
+      )
+    )
+  )
   (symbol (lib_id "Device:C") (at 110.49 77.47 90) (unit 1)
     (in_bom yes) (on_board yes) (dnp no) (fields_autoplaced)
@@
         (path "/76d5dda2-c124-4f87-b6ec-acef9f17eff7"
           (reference "C1") (unit 1)
+        )
+      )
+    )
+  )
+  (symbol (lib_id "Device:C") (at 135.89 88.9 90) (unit 1)
+    (in_bom yes) (on_board yes) (dnp no) (fields_autoplaced)
+    (property "Reference" "C2" (at 135.89 81.28 90)
+      (effects (font (size 1.27 1.27)))
+    )
+    (property "Value" "C" (at 135.89 83.82 90)
+      (effects (font (size 1.27 1.27)))
+    )
+    (property "Footprint" "" (at 139.7 87.9348 0)
+      (effects (font (size 1.27 1.27)) hide)
+    )
+    (property "Datasheet" "~" (at 135.89 88.9 0)
+      (effects (font (size 1.27 1.27)) hide)
+    )
+    (pin "1")
+    (pin "2")
+    (instances
+      (project "555_pwm"
+        (path "/76d5dda2-c124-4f87-b6ec-acef9f17eff7"
+          (reference "C2") (unit 1)
         )
       )
@@
         )
       )
+    )
+  )
+  (symbol (lib_id "power:GND") (at 127 99.06 0) (unit 1)
+    (in_bom yes) (on_board yes) (dnp no) (fields_autoplaced)
+    (property "Reference" "#PWR02" (at 127 105.41 0)
+      (effects (font (size 1.27 1.27)) hide)
+    )
+    (property "Value" "GND" (at 127 104.14 0)
+      (effects (font (size 1.27 1.27)))
+    )
+    (property "Footprint" "" (at 127 99.06 0)
+      (effects (font (size 1.27 1.27)) hide)
+    )
+    (property "Datasheet" "" (at 127 99.06 0)
+      (effects (font (size 1.27 1.27)) hide)
+    )
+    (pin "1")
+    (instances
+      (project "555_pwm"
+        (path "/76d5dda2-c124-4f87-b6ec-acef9f17eff7"
+          (reference "#PWR02") (unit 1)
+        )
+      )

Commit message: a
Parts:
- added C3: C, symbol Device:C
- added D1, D2, D3, D4, D5, D6, D7, D8: LED, symbol Device:LED
- added D10, D11, D12, D13, D14, D15, D16, D9: D, symbol Device:D
- added J1, J2: Conn_01x08_Pin, symbol Connector:Conn_01x08_Pin
- added R10, R3, R4, R5, R6, R7, R8, R9: R, symbol Device:R
- added U2: 74HC595, symbol 74xx:74HC595
- added U3, U4: 74LS04, symbol 74xx:74LS04
Connections:
- net +5V: now also C3.1, U2.10 (~{SRCLR}), U2.16 (VCC)
- net GND: now also C1.1, C3.2, J2.1 (Pin_1), J2.2 (Pin_2), J2.3 (Pin_3), J2.4 (Pin_4), J2.5 (Pin_5), J2.6 (Pin_6), J2.7 (Pin_7), J2.8 (Pin_8), U2.13 (~{OE}), U2.8 (GND)
- net at C2.2, R2.2, U1.2 (TR)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: no longer C1.1
- net at U1.3 (Q): now also U2.11 (SRCLK), U4.1
- new net: D4.1 (K), R6.1
- new net: J1.5 (Pin_5), R6.2
- new net: D8.1 (K), R10.1
- new net: D8.2 (A), D9.2 (A), U2.7 (QH)
- new net: D10.1 (K), D11.1 (K), D12.1 (K), D13.1 (K), D14.1 (K), D15.1 (K), D16.1 (K), D9.1 (K), U3.1
- new net: U2.14 (SER), U3.2
- new net: D1.1 (K), R3.1
- new net: D1.2 (A), D16.2 (A), U2.15 (QA)
- new net: D3.1 (K), R5.1
- new net: D14.2 (A), D3.2 (A), U2.2 (QC)
- new net: D2.1 (K), R4.1
- new net: J1.7 (Pin_7), R4.2
- new net: D5.1 (K), R7.1
- new net: J1.4 (Pin_4), R7.2
- new net: D13.2 (A), D4.2 (A), U2.3 (QD)
- new net: D15.2 (A), D2.2 (A), U2.1 (QB)
- new net: D12.2 (A), D5.2 (A), U2.4 (QE)
- new net: J1.1 (Pin_1), R10.2
- new net: J1.2 (Pin_2), R9.2
- new net: J1.3 (Pin_3), R8.2
- new net: J1.6 (Pin_6), R5.2
- new net: J1.8 (Pin_8), R3.2
- new net: U2.12 (RCLK), U4.2
- new net: D10.2 (A), D7.2 (A), U2.6 (QG)
- new net: D7.1 (K), R9.1
- new net: D11.2 (A), D6.2 (A), U2.5 (QF)
- new net: D6.1 (K), R8.1
Other:
- moved on the sheet: C1, C2, R1, R2, U1
