File: router/RJ45.kicad_sch (KiCad schematic)
At the start: 0 parts

Commit message: new symbols
Parts:
- added D1, D2, D3, D4: TPD4E05U06DQAR, DQA(R-PUSON-N10), symbol TPD4E05U06DQAR:TPD4E05U06DQAR
- added J1: TMJG26945AENL, TMJG26945AENL, symbol TMJG26945AENL:TMJG26945AENL
- added R1, R2, R3, R4: 680, symbol Device:R
Connections:
- new net: J1.A13 (A_YELLOW_1), R2.2
- new net: J1.B13 (A_YELLOW_2), R3.2
- new net: J1.A11 (A_GREEN_1), R1.2
- new net: J1.B11 (A_GREEN_2), R4.2
- new net +3V3: R1.1, R2.1, R3.1, R4.1
- new net ETH1_LEDG: J1.A12 (K_GREEN_1)
- new net ETH1_LEDY: J1.A14 (K_YELLOW_1)
- new net ETH2_LEDG: J1.B12 (K_GREEN_2)
- new net ETH2_LEDY: J1.B14 (K_YELLOW_2)
- no-connect marks 0 -> 4

Commit message: huge cock
Parts:
- renumbered J1 to J2, R3 to R10, R2 to R8, R1 to R9
Connections:
- net ETH2_MDIP2: now reaches D2.1 (D1+)
- net ETH2_MDIP2: now also D2.10 (NC_4), J2.A6 (TD2+_1)
- net ETH2_MDIN2: now reaches D2.2 (D1-)
- net ETH2_MDIN2: now also D2.9 (NC_3), J2.A7 (TD2-_1)
- net GND: now reaches D2.3 (GND_1)
- net GND: now also D1.3 (GND_1), D1.8 (GND_2), D2.8 (GND_2), D3.3 (GND_1), D3.8 (GND_2), D4.3 (GND_1), D4.8 (GND_2)
- net ETH2_MDIP3: now reaches D2.4 (D2+)
- net ETH2_MDIP3: now also D2.7 (NC_2), J2.A8 (TD3+_1)
- net ETH2_MDIN3: now reaches D2.5 (D2-)
- net ETH2_MDIN3: now also D2.6 (NC_1), J2.A9 (TD3-_1)
- net ETH2_MDIP0: now reaches J2.A2 (TD0+_1)
- net ETH2_MDIP0: now also D1.1 (D1+), D1.10 (NC_4)
- net ETH2_MDIN0: now reaches J2.A3 (TD0-_1)
- net ETH2_MDIN0: now also D1.2 (D1-), D1.9 (NC_3)
- net ETH2_MDIP1: now reaches J2.A4 (TD1+_1)
- net ETH2_MDIP1: now also D1.4 (D2+), D1.7 (NC_2)
- net ETH2_MDIN1: now reaches J2.A5 (TD1-_1)
- net ETH2_MDIN1: now also D1.5 (D2-), D1.6 (NC_1)
- net ETH1_DIP0: now reaches J2.B2 (TD0+_2)
- net ETH1_DIP0: now also D3.1 (D1+), D3.10 (NC_4)
- net ETH1_DIN0: now reaches J2.B3 (TD0-_2)
- net ETH1_DIN0: now also D3.2 (D1-), D3.9 (NC_3)
- net ETH1_MDIP1: now reaches J2.B4 (TD1+_2)
- net ETH1_MDIP1: now also D3.4 (D2+), D3.7 (NC_2)
- net ETH1_MDIN1: now reaches J2.B5 (TD1-_2)
- net ETH1_MDIN1: now also D3.5 (D2-), D3.6 (NC_1)
- net ETH1_MDIP2: now reaches J2.B6 (TD2+_2)
- net ETH1_MDIP2: now also D4.1 (D1+), D4.10 (NC_4)
- net ETH1_MDIN2: now reaches J2.B7 (TD2-_2)
- net ETH1_MDIN2: now also D4.2 (D1-), D4.9 (NC_3)
- net ETH1_MDIP3: now reaches J2.B8 (TD3+_2)
- net ETH1_MDIP3: now also D4.4 (D2+), D4.7 (NC_2)
- net ETH1_MDIN3: now reaches J2.B9 (TD3-_2)
- net ETH1_MDIN3: now also D4.5 (D2-), D4.6 (NC_1)
- net GNDPWR: now reaches J2.MH1
- net GNDPWR: now also J2.MH2, J2.MH3
Other:
- moved on the sheet: D1
