File: router/router.kicad_sch (KiCad schematic)
At the start: 17 parts, among them J1 UART interface

Commit message: huge cock
Other:
- added sheet LAN7800 (LAN7800.kicad_sch)
Changed lines of the file:
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@@
     )
   )
-  (sheet (at 297.18 24.13) (size 66.04 67.31) (fields_autoplaced)
+  (sheet (at 299.72 25.4) (size 26.67 26.67) (fields_autoplaced)
     (stroke (width 0.1524) (type solid))
     (fill (color 0 0 0 0.0000))
-    (property "Sheetname" "RJ45" (at 297.18 23.4184 0)
+    (property "Sheetname" "RJ45" (at 299.72 24.6884 0)
       (effects (font (size 1.27 1.27)) (justify left bottom))
     )
-    (property "Sheetfile" "RJ45.kicad_sch" (at 297.18 92.0246 0)
+    (property "Sheetfile" "RJ45.kicad_sch" (at 299.72 52.6546 0)
       (effects (font (size 1.27 1.27)) (justify left top))
     )
@@
       )
     )
+  )
+  (sheet (at 330.2 25.4) (size 26.67 26.67) (fields_autoplaced)
+    (stroke (width 0.1524) (type solid))
+    (fill (color 0 0 0 0.0000))
+    (property "Sheetname" "LAN7800" (at 330.2 24.6884 0)
+      (effects (font (size 1.27 1.27)) (justify left bottom))
+    )
+    (property "Sheetfile" "LAN7800.kicad_sch" (at 330.2 52.6546 0)
+      (effects (font (size 1.27 1.27)) (justify left top))
+    )
+    (instances
+      (project "router"
+        (path "/0c416362-cc48-4bc2-9846-eef228bc2951" (page "3"))
+      )
+    )
